File: KicadSMD/PiRTO_cart.kicad_pcb (KiCad board)
At the start: 2 copper layers, 58.2 x 77.5 mm, 11 parts, among them J1 2x22 card edge connector, J3 Micro_SD_Card, U1 74LVC245, U2 74LVC245, U3 74LVC245, U4 74LVC245

Commit message: Add files via upload
Parts:
- added JP1: 3v3, Jumper:SolderJumper-2_P1.3mm_Open_Pad1.0x1.5mm, F.Cu at (118.7, 119.4)
- added JP2: Gnd, Jumper:SolderJumper-2_P1.3mm_Open_Pad1.0x1.5mm, F.Cu at (111.1, 119.4)
- added JP3: Shield, Jumper:SolderJumper-2_P1.3mm_Open_Pad1.0x1.5mm, F.Cu at (108.6, 109.2)
Connections:
- J3 pad 4: +3.3V -> Net-(J3-VDD)
- J3 pad 6: GND -> Net-(J3-VSS)
- J3 pad 9: GND -> Net-(J3-SHIELD)
Routing:
- net GND: track 443.5 -> 408.0 mm
- net +3.3V: track 111.8 -> 139.1 mm, vias 4 -> 3
- net Net-(J3-VDD): track 0.00 -> 23.1 mm
- net D7: track 38.4 -> 61.0 mm
- net BC1: track 42.7 -> 60.6 mm, vias 2 -> 1
- net Net-(J3-VSS): track 0.00 -> 16.5 mm
- net D6: track 37.0 -> 49.1 mm, vias 1 -> 0
- net D12: track 44.9 -> 32.8 mm, vias 1 -> 0
- net MISO: track 47.1 -> 55.9 mm
- net D5: track 53.6 -> 45.7 mm, vias 0 -> 1
- net Net-(J3-SHIELD): track 0.00 -> 6.99 mm
- net D2: track 26.9 -> 32.2 mm
- net BC2: track 47.8 -> 43.8 mm, vias 2 -> 0
- net RST: track 48.0 -> 45.3 mm
- net bdir': track 46.0 -> 48.6 mm
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Other:
- board text added: "solder all jumper"
